File: CFR_module_v1.kicad_pcb (KiCad board)
At the start: 2 copper layers, 39 parts, among them J6 Conn_01x20, J7 Conn_01x03, J8 Conn_01x20

Commit message: Modifs
Parts:
- removed A1, A2: Conn_01x04_Pin, Connector_PinHeader_2.54mm:PinHeader_1x04_P2.54mm_Vertical
- removed A3, A4: Conn_01x01_Pin, Connector_PinHeader_2.54mm:PinHeader_1x01_P2.54mm_Vertical
- removed ALM1: Conn_01x04_Pin, Connector_JST:JST_EH_B4B-EH-A_1x04_P2.50mm_Vertical
- removed C1, C2: 100uF/35V, Capacitor_THT:CP_Radial_D6.3mm_P2.50mm
- removed D1, D2, D3, D4: D, Diode_THT:D_DO-41_SOD81_P7.62mm_Horizontal
- removed D5: D_Schottky, Diode_THT:D_DO-41_SOD81_P10.16mm_Horizontal
- removed DR1, DR2: Pololu_Breakout, Custom:Pololu_Breakout-16_15.2x20.3mm_Better_Silkscreen
- removed J6, J8: Conn_01x20, Connector_PinSocket_2.54mm:PinSocket_1x20_P2.54mm_Vertical
- removed J7: Conn_01x03, Connector_PinSocket_2.54mm:PinSocket_1x03_P2.54mm_Vertical
- removed JP1, JP3, JP5, JP6, JP7, JP9: Conn_01x03_Pin, Connector_PinSocket_2.54mm:PinSocket_1x03_P2.54mm_Vertical
- removed JP10, JP2, JP4, JP8: Conn_01x02_Pin, Connector_PinSocket_2.54mm:PinSocket_1x02_P2.54mm_Vertical
- removed MF1, MF2: NMOS, Package_TO_SOT_THT:TO-220-3_Vertical
- removed MOT1, MOT2, S1, S2: Conn_01x04_Pin, Connector_PinSocket_2.54mm:PinSocket_1x04_P2.54mm_Vertical
- removed Pico0: RaspberryPi_Pico, Module:RaspberryPi_Pico_Common_Unspecified
- removed R1: 1k, Resistor_THT:R_Axial_DIN0207_L6.3mm_D2.5mm_P7.62mm_Horizontal
- removed R2, R4: 10k, Resistor_THT:R_Axial_DIN0207_L6.3mm_D2.5mm_P7.62mm_Horizontal
- removed R3, R5: 330, Resistor_THT:R_Axial_DIN0207_L6.3mm_D2.5mm_P7.62mm_Horizontal

Commit message: v1 du schematics, debut de pcb
Parts:
- added ALM1: Conn_01x02, Connector_AMASS:AMASS_XT30U-F_1x02_P5.0mm_Vertical, F.Cu at (77.0, 159.0)
- added ALM2: Conn_01x02, Connector_AMASS:AMASS_XT30U-F_1x02_P5.0mm_Vertical, F.Cu at (86.5, 159.0)
- added ALM3: Conn_01x02, Connector_AMASS:AMASS_XT30U-F_1x02_P5.0mm_Vertical, F.Cu at (96.0, 159.0)
- added ALM4: Conn_01x02, Connector_AMASS:AMASS_XT30U-F_1x02_P5.0mm_Vertical, F.Cu at (105.5, 159.0)
- added C1: C_Polarized, Capacitor_SMD:CP_Elec_10x10.5, F.Cu at (84.0, 147.8)
- added C2: C_Polarized, Capacitor_SMD:CP_Elec_8x10, F.Cu at (95.5, 149.2)
- added C3: C_Polarized, Capacitor_SMD:CP_Elec_6.3x5.8, F.Cu at (104.5, 150.3)
- added C4: 100uF/35V, Capacitor_THT:CP_Radial_D6.3mm_P2.50mm, F.Cu at (147.5, 75.0)
- added C5: 100uF/35V, Capacitor_THT:CP_Radial_D6.3mm_P2.50mm, F.Cu at (147.5, 97.0)
- added C6: 100uF/35V, Capacitor_THT:CP_Radial_D6.3mm_P2.50mm, F.Cu at (147.5, 120.5)
- added D1: D, Diode_SMD:D_SMA_Handsoldering, F.Cu at (40.5, 74.4)
- added D2: D, Diode_SMD:D_SMA_Handsoldering, F.Cu at (82.5, 126.5)
- added D3: D, Diode_SMD:D_SMA_Handsoldering, F.Cu at (186.7, 71.2)
- added D4: D, Diode_SMD:D_SMA_Handsoldering, F.Cu at (186.7, 75.8)
- added D5: D, Diode_SMD:D_SMA_Handsoldering, F.Cu at (185.0, 83.5)
- added D6: D_Schottky, Diode_SMD:D_SOD-123, F.Cu at (85.5, 70.0)
- added DBG1: Conn_01x02_Socket, Connector_PinHeader_2.54mm:PinHeader_1x02_P2.54mm_Vertical, F.Cu at (50.0, 70.0)
- added DR1: Pololu_Breakout, Custom:Pololu_Breakout-16_15.2x20.3mm_Better_Silkscreen, F.Cu at (142.5, 59.6)
- added DR2: Pololu_Breakout, Custom:Pololu_Breakout-16_15.2x20.3mm_Better_Silkscreen, F.Cu at (142.5, 81.7)
- added DR3: Pololu_Breakout, Custom:Pololu_Breakout-16_15.2x20.3mm_Better_Silkscreen, F.Cu at (142.5, 105.3)
- added F1: Fuse, Fuse:Fuse_1206_3216Metric_Pad1.42x1.75mm_HandSolder, F.Cu at (78.5, 154.5)
- added F2: Fuse, Fuse:Fuse_1206_3216Metric_Pad1.42x1.75mm_HandSolder, F.Cu at (91.0, 155.0)
- added F3: Fuse, Fuse:Fuse_1206_3216Metric_Pad1.42x1.75mm_HandSolder, F.Cu at (100.5, 155.0)
- added IO1: Conn_01x04, Connector_JST:JST_PH_B4B-PH-K_1x04_P2.00mm_Vertical, F.Cu at (36.5, 73.4)
- added IO2: Conn_01x04, Connector_JST:JST_PH_B4B-PH-K_1x04_P2.00mm_Vertical, F.Cu at (86.5, 127.5)
- added IO3: Conn_01x03, Connector_JST:JST_PH_B3B-PH-K_1x03_P2.00mm_Vertical, F.Cu at (164.3, 113.5)
- added IO4: Conn_01x03, Connector_JST:JST_PH_B3B-PH-K_1x03_P2.00mm_Vertical, F.Cu at (164.3, 120.0)
- added IO5: Conn_01x03, Connector_JST:JST_PH_B3B-PH-K_1x03_P2.00mm_Vertical, F.Cu at (164.3, 126.6)
- added J1: Conn_01x20, Connector_PinSocket_2.54mm:PinSocket_1x20_P2.54mm_Vertical, F.Cu at (54.0, 67.6)
- added J2: Conn_01x20, Connector_PinSocket_2.54mm:PinSocket_1x20_P2.54mm_Vertical, F.Cu at (81.0, 67.5)
- added JP1: Jumper_3_Bridged12, Connector_PinHeader_2.54mm:PinHeader_1x03_P2.54mm_Vertical, F.Cu at (173.6, 113.0)
- added JP10: Jumper_3_Bridged12, Connector_PinHeader_2.54mm:PinHeader_1x03_P2.54mm_Vertical, F.Cu at (178.2, 122.7)
- added JP11: Jumper_3_Bridged12, Connector_PinHeader_2.54mm:PinHeader_1x03_P2.54mm_Vertical, F.Cu at (182.8, 122.7)
- added JP12: Jumper_3_Bridged12, Connector_PinHeader_2.54mm:PinHeader_1x03_P2.54mm_Vertical, F.Cu at (192.0, 122.7)
- added JP13: Jumper_3_Bridged12, Connector_PinHeader_2.54mm:PinHeader_1x03_P2.54mm_Vertical, F.Cu at (103.5, 138.0)
- added JP14: Jumper_3_Bridged12, Connector_PinHeader_2.54mm:PinHeader_1x03_P2.54mm_Vertical, F.Cu at (103.5, 141.5)
- added JP2: Jumper_3_Bridged12, Connector_PinHeader_2.54mm:PinHeader_1x03_P2.54mm_Vertical, F.Cu at (178.2, 113.0)
- added JP3: Jumper_3_Bridged12, Connector_PinHeader_2.54mm:PinHeader_1x03_P2.54mm_Vertical, F.Cu at (182.8, 113.0)
- added JP4: Jumper_3_Bridged12, Connector_PinHeader_2.54mm:PinHeader_1x03_P2.54mm_Vertical, F.Cu at (187.4, 113.0)
- added JP5: Jumper_3_Bridged12, Connector_PinHeader_2.54mm:PinHeader_1x03_P2.54mm_Vertical, F.Cu at (192.0, 113.0)
- added JP6: Jumper_3_Bridged12, Connector_PinHeader_2.54mm:PinHeader_1x03_P2.54mm_Vertical, F.Cu at (217.0, 89.5)
- added JP7: Jumper_3_Bridged12, Connector_PinHeader_2.54mm:PinHeader_1x03_P2.54mm_Vertical, F.Cu at (44.5, 79.5)
- added JP8: Jumper_3_Bridged12, Connector_PinHeader_2.54mm:PinHeader_1x03_P2.54mm_Vertical, F.Cu at (78.5, 121.5)
- added JP9: Jumper_3_Bridged12, Connector_PinHeader_2.54mm:PinHeader_1x03_P2.54mm_Vertical, F.Cu at (173.6, 122.7)
- added MOT1: Conn_01x04, Connector_PinHeader_2.54mm:PinHeader_1x04_P2.54mm_Vertical, F.Cu at (139.0, 72.3)
- added MOT2: Conn_01x04, Connector_PinHeader_2.54mm:PinHeader_1x04_P2.54mm_Vertical, F.Cu at (139.0, 94.4)
- added MOT3: Conn_01x04, Connector_PinHeader_2.54mm:PinHeader_1x04_P2.54mm_Vertical, F.Cu at (139.0, 118.0)
- added Pico0: RaspberryPi_Pico, Module:RaspberryPi_Pico_Common_Unspecified, F.Cu at (67.5, 91.6)
- added R1: 1k, Resistor_SMD:R_0805_2012Metric_Pad1.20x1.40mm_HandSolder, F.Cu at (207.0, 84.0)
- added R2: 1k, Resistor_SMD:R_0805_2012Metric_Pad1.20x1.40mm_HandSolder, F.Cu at (207.0, 86.5)
- added R3: 1k, Resistor_SMD:R_0805_2012Metric_Pad1.20x1.40mm_HandSolder, F.Cu at (207.0, 89.5)
